Commit message: host: ollie_description: add sensors
adds sensor in urdf
add fake_ollie_core.py sensor fake data

File: host/ros2_ws/src/ollie_description/urdf/ollie.urdf (robot description, URDF)
Before this commit: robot ollie, 5 links, 4 joints
Links:
- added link left_ultrasonic_link; visual box size=0.01 0.04 0.02
- added link right_ultrasonic_link; visual box size=0.01 0.04 0.02
Joints:
- added joint left_ultrasonic_joint: type fixed, parent base_link, child left_ultrasonic_link, origin xyz=0.12 0.05 -0.0525 rpy=0 0 0
- added joint right_ultrasonic_joint: type fixed, parent base_link, child right_ultrasonic_link, origin xyz=0.12 -0.05 -0.0525 rpy=0 0 0

Commit message: host: lidar: setup lib and urdf
add lidar urdf description.
build lidar driver.

File: host/ros2_ws/src/ollie_description/urdf/ollie.urdf (robot description, URDF)
Before this commit: robot ollie, 7 links, 6 joints
Links:
- removed link lidar_link
- added link base_laser; visual cylinder length=0.04 radius=0.02
Joints:
- joint lidar_joint: child lidar_link -> base_laser

Commit message: host: fix lidar and sonic positions in URDF
fixed position.

File: host/ros2_ws/src/ollie_description/urdf/ollie.urdf (robot description, URDF)
Before this commit: robot ollie, 7 links, 6 joints
Links:
- link base_laser: geometry visual cylinder length=0.02 radius=0.02
- link base_link: geometry visual box size=0.26 0.16 0.055
Joints:
- joint left_ultrasonic_joint: origin xyz=0.12 0.05 -0.0525 rpy=0 0 0 -> xyz=0.095 0.04 -0.0525 rpy=0 0 0.1745
- joint left_wheel_joint: type continuous -> fixed
- joint lidar_joint: origin xyz=0.05 0 0.0275 rpy=0 0 0 -> xyz=0.015 -0.005 0.0425 rpy=0 0 -0.0873
- joint right_ultrasonic_joint: origin xyz=0.12 -0.05 -0.0525 rpy=0 0 0 -> xyz=0.095 -0.04 -0.0525 rpy=0 0 -0.1745
- joint right_wheel_joint: type continuous -> fixed
