Commit message: urdf: update the new urdf
Updated to cylinder type.

File: host_2404/ros2_ws/src/ollie_description/urdf/ollie.urdf (robot description, URDF)
Before this commit: robot ollie, 7 links, 6 joints
Links:
- added link base_footprint
- link base_link: geometry collision cylinder length=0.10 radius=0.135; visual cylinder length=0.10 radius=0.135
- link caster_wheel: geometry collision sphere radius=0.0075; visual sphere radius=0.0075
- link left_wheel: geometry collision cylinder length=0.014 radius=0.0325; visual cylinder length=0.014 radius=0.0325
- link right_wheel: geometry collision cylinder length=0.014 radius=0.0325; visual cylinder length=0.014 radius=0.0325
Joints:
- added joint base_footprint_joint: type fixed, parent base_footprint, child base_link, origin xyz=0 0 0.0105 rpy=0 0 0
- joint caster_joint: origin xyz=-0.07 0 -0.0625 rpy=0 0 0 -> xyz=0.095 0 -0.003 rpy=0 0 0
- joint left_ultrasonic_joint: origin xyz=0.095 0.04 -0.0525 rpy=0 0 0.1745 -> xyz=0.11 0.045 0.0295 rpy=0 0 0.3882
- joint left_wheel_joint: origin xyz=0.025 0.068 -0.0395 rpy=0 0 0 -> xyz=-0.005 0.095 0.022 rpy=0 0 0; type fixed -> continuous
- joint lidar_joint: origin xyz=0.015 -0.005 0.0425 rpy=0 0 -0.0873 -> xyz=0.095 0 0.0695 rpy=0 0 0
- joint right_ultrasonic_joint: origin xyz=0.095 -0.04 -0.0525 rpy=0 0 -0.1745 -> xyz=0.11 -0.045 0.0295 rpy=0 0 -0.3882
- joint right_wheel_joint: origin xyz=0.025 -0.068 -0.0395 rpy=0 0 0 -> xyz=-0.005 -0.095 0.022 rpy=0 0 0; type fixed -> continuous
